File: VFD.kicad_pcb (KiCad board)
At the start: 2 copper layers, 39 parts, among them J1 Conn_01x06, J2 Screw_Terminal_01x02, J3 Screw_Terminal_01x02, J4 Conn_01x04, Q1 IPW60R037P7, Q2 IPW60R037P7, Q3 IPW60R037P7, Q4 IPW60R037P7, U1 2ED2182S06F, U2 2ED2182S06F

Commit message: 1
Parts:
- removed C15: 2200u, Capacitor_THT:CP_Radial_D30.0mm_P10.00mm_SnapIn
- D4: value D_Bridge_+AA- -> D_Bridge_-AA+
- moved J2 183.5 mm to (97.5, 27.4), turned to 180 degrees
- moved D4 162.5 mm to (107.6, 40.6)
- moved U2 141.1 mm to (197.2, 56.4), turned to 90 degrees
- moved F1 127.7 mm to (93.0, 71.1), turned to 90 degrees
- moved PS1 120.5 mm to (103.6, 58.2)
- moved C5 118.9 mm to (188.0, 94.0)
- moved C11 112.5 mm to (167.6, 24.1), turned to 90 degrees
- moved C13 111.1 mm to (201.2, 24.1), turned to 90 degrees
- moved J4 109.7 mm to (182.6, 75.2)
- moved C10 109.6 mm to (134.1, 24.1), turned to 90 degrees
- moved C7 108.4 mm to (172.2, 90.2)
- moved C14 103.6 mm to (190.4, 57.4), turned to 180 degrees
- moved C12 102.2 mm to (191.4, 53.3), turned to 180 degrees
- moved J1 92.5 mm to (161.0, 75.9)
- moved C17 88.2 mm to (203.1, 53.3)
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Connections:
- D4 pad 1: VCC -> GND
- D4 pad 4: GND -> VCC
Routing:
- net NEUT: track 0.00 -> 25.1 mm
- net Net-(D6-Pad1): track 0.00 -> 21.5 mm
- net VOUT_B: track 18.0 -> 0.00 mm
- net VOUT_A: track 17.8 -> 0.00 mm
- net Net-(D6-Pad2): track 0.00 -> 15.6 mm
- net Net-(D5-Pad2): track 0.00 -> 12.3 mm
- net Net-(C12-Pad1): track 0.00 -> 11.6 mm
- net Net-(D5-Pad1): track 0.00 -> 8.63 mm
- net +12V: track 7.25 -> 14.5 mm
- net Net-(C3-Pad1): track 7.25 -> 11.6 mm
- net Net-(D3-Pad2): track 14.0 -> 15.6 mm
- added copper zone on B.Cu, net GND
- added copper zone on F.Cu, net LINE
- added copper zone on F.Cu, net NEUT
- added copper zone on F.Cu, net Net-(D4-Pad2)
- added copper zone on F.Cu, net VCC
- removed copper zone on F.Cu, net VOUT_A

Commit message: 1
Parts:
- added J5: Screw_Terminal_01x01, Connector_Wire:SolderWire-1.5sqmm_1x01_D1.7mm_OD3mm, F.Cu at (178.3, 96.1)
- J3: value Screw_Terminal_01x02 -> Screw_Terminal_01x01; footprint Connector_Wire:SolderWire-1.5sqmm_1x02_P6mm_D1.7mm_OD3mm -> Connector_Wire:SolderWire-1.5sqmm_1x01_D1.7mm_OD3mm
- moved J3 127.3 mm to (149.7, 96.1)
- moved PS1 62.1 mm to (99.8, 120.2)
- moved R1 62.1 mm to (149.6, 110.6)
- moved R3 62.1 mm to (188.7, 110.6)
- moved U1 62.1 mm to (154.3, 118.4)
- moved U2 62.1 mm to (193.4, 118.4)
- moved C1 62.1 mm to (160.2, 115.3)
- moved C10 62.1 mm to (130.3, 86.1)
- moved C11 62.1 mm to (163.8, 86.1)
- moved C12 62.1 mm to (187.6, 115.3)
- moved C13 62.1 mm to (197.4, 86.1)
- moved C17 62.1 mm to (199.3, 115.3)
- moved C4 62.1 mm to (148.4, 115.3)
- moved D3 62.1 mm to (168.5, 113.9)
- moved D4 62.1 mm to (103.8, 102.6)
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Connections:
- C5 pad 2: Net-(C5-Pad2) -> GND
- C7 pad 2: Net-(C5-Pad2) -> GND
- J3 pad 1: VOUT_B -> VOUT_A
- PS1 pad 3: Net-(C5-Pad2) -> GND
Routing:
- net +12V: track 14.5 -> 113.8 mm, vias 0 -> 5
- net DRV_B: track 0.00 -> 43.4 mm, vias 0 -> 2
- net DRV_A: track 0.00 -> 41.0 mm, vias 0 -> 3
- net DRV_D: track 0.00 -> 33.0 mm, vias 0 -> 2
- net VOUT_B: track 0.00 -> 28.4 mm, vias 0 -> 28
- net VOUT_A: track 0.00 -> 28.4 mm, vias 0 -> 11
- net DRV_C: track 0.00 -> 28.0 mm, vias 0 -> 2
- net GND: vias 0 -> 100
- added copper zone on F.Cu, net GND
- added copper zone on B.Cu, net VOUT_A
- added copper zone on F.Cu, net VOUT_A
- added copper zone on B.Cu, net VOUT_B
- added copper zone on F.Cu, net VOUT_B

Commit message: 1
Other:
- board outline added: 127.3 x 68.8 mm

Commit message: 1
Routing:
- net GND: vias 100 -> 99
Other:
- board size 127.3 x 68.8 mm -> 128.3 x 70.4 mm
- net class HV added: clearance 1, trace_width 0.25, via_dia 0.8, via_drill 0.4

Commit message: 1
Parts:
- Q1, Q2, Q3, Q4: value IPW60R037P7 -> IPW60R060P7
