File: VFD.kicad_pcb (KiCad board)
At the start: 2 copper layers, 128.3 x 70.4 mm, 39 parts, among them J1 Conn_01x06, J2 Screw_Terminal_01x02, J3 Screw_Terminal_01x01, J4 Conn_01x04, J5 Screw_Terminal_01x01, Q1 IPW60R060P7, Q2 IPW60R060P7, Q3 IPW60R060P7, Q4 IPW60R060P7, U1 2ED2182S06F, U2 2ED2182S06F

Commit message: Update Gate Resistor Values
Parts:
- Q1, Q2, Q3, Q4: value IPW60R060P7 -> IPW60R037CSFD
- R1, R2, R3, R4: value 0 -> 10

Commit message: Fix Issues
Parts:
- added C15: 1u, Capacitor_THT:C_Rect_L19.0mm_W8.0mm_P15.00mm_MKS4, F.Cu at (109.7, 70.1)
- added C8: 1u, Capacitor_THT:C_Rect_L19.0mm_W8.0mm_P15.00mm_MKS4, F.Cu at (109.7, 80.8)
- added REF**: MountingHole_2.7mm_M2.5, MountingHole:MountingHole_2.7mm_M2.5, F.Cu at (210.6, 133.1)
- added REF**: MountingHole_2.7mm_M2.5, MountingHole:MountingHole_2.7mm_M2.5, F.Cu at (210.6, 67.8)
- added REF**: MountingHole_2.7mm_M2.5, MountingHole:MountingHole_2.7mm_M2.5, F.Cu at (87.4, 67.8)
Routing:
- net GND: vias 99 -> 83

Commit message: 1
Other:
- net class Default removed
- net class HV removed
